File: hardware/open-circuit.brd (EAGLE design)
At the start: 90.2 x 40.6 mm, 75 parts, among them IC1 PIC16F1825SO14, IC2 74HC595D, IC3 MCP4728_QUAD_DAC, IC4 LM324D, IC5 REG1117, IC6 LM27675M5_CHARGEPUMP

Commit message: updates
Parts:
- removed R10, R11, R7, R8: (no value), rcl:R0805
Connections:
- removed net N$29: R11.2, VELA.4
- removed net N$30: NOTA.4, R8.2
- removed net N$31: NOTB.4, R7.2
- removed net N$32: R10.2, VELB.4
- net N$2: now also VELA.4; no longer R11.1
- net N$3: now also NOTA.4; no longer R8.1
- net N$4: now also NOTB.4; no longer R7.1
- net N$5: now also VELB.4; no longer R10.1
Routing:
- net N$32: track 4.14 -> 0.00 mm
- net N$31: track 4.14 -> 0.00 mm
- net N$30: track 4.14 -> 0.00 mm
- net N$29: track 4.14 -> 0.00 mm
- net N$5: track 32.3 -> 30.8 mm
- net N$3: track 24.2 -> 22.7 mm
- net N$4: track 29.0 -> 27.7 mm
- net N$2: track 21.1 -> 22.3 mm
Changed lines of the file:
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@@
 <attribute name="NAME" x="67.183" y="47.371" size="1.27" layer="25" rot="R180"/>
-</element>
-<element name="R8" library="rcl" package="R0805" value="" x="53.34" y="64.77" smashed="yes" rot="R180">
-<attribute name="NAME" x="55.372" y="65.913" size="1.27" layer="25" rot="R270"/>
-<attribute name="VALUE" x="53.975" y="67.31" size="1.27" layer="27" rot="R180"/>
-</element>
-<element name="R11" library="rcl" package="R0805" value="" x="53.34" y="52.07" smashed="yes" rot="R180">
-<attribute name="NAME" x="55.372" y="53.594" size="1.27" layer="25" rot="R270"/>
-<attribute name="VALUE" x="53.975" y="54.61" size="1.27" layer="27" rot="R180"/>
-</element>
-<element name="R7" library="rcl" package="R0805" value="" x="40.64" y="64.77" smashed="yes" rot="R180">
-<attribute name="NAME" x="45.085" y="65.405" size="1.27" layer="25" rot="R180"/>
-<attribute name="VALUE" x="41.275" y="67.31" size="1.27" layer="27" rot="R180"/>
-</element>
-<element name="R10" library="rcl" package="R0805" value="" x="40.64" y="52.07" smashed="yes" rot="R180">
-<attribute name="NAME" x="46.101" y="52.705" size="1.27" layer="25" rot="R180"/>
-<attribute name="VALUE" x="41.275" y="54.61" size="1.27" layer="27" rot="R180"/>
 </element>
 <element name="R27" library="rcl" package="R0805" value="" x="71.12" y="49.53" smashed="yes" rot="R270">
@@
 <wire x1="70.8" y1="48.26" x2="71.12" y2="48.58" width="0.4064" layer="1"/>
 <contactref element="IC4" pad="1"/>
-<contactref element="R11" pad="1"/>
 <wire x1="70.8" y1="48.26" x2="68.64" y2="48.26" width="0.4064" layer="1"/>
 <wire x1="68.64" y1="48.26" x2="67.31" y2="48.26" width="0.4064" layer="1"/>
@@
 <wire x1="56.515" y1="49.022" x2="54.229" y2="51.308" width="0.4064" layer="1"/>
 <wire x1="54.229" y1="51.308" x2="54.229" y2="52.009" width="0.4064" layer="1"/>
-<wire x1="54.229" y1="52.009" x2="54.29" y2="52.07" width="0.4064" layer="1"/>
+<contactref element="VELA" pad="4"/>
+<wire x1="52.39" y1="54.87" x2="53.34" y2="55.82" width="0.4064" layer="1"/>
+<wire x1="54.229" y1="52.009" x2="52.39" y2="54.87" width="0" layer="19" extent="1-1"/>
 </signal>
 <signal name="N$3">
 <contactref element="R22" pad="2"/>
 <contactref element="IC4" pad="7"/>
-<contactref element="R8" pad="1"/>
 <wire x1="68.64" y1="55.88" x2="70.8" y2="55.88" width="0.4064" layer="1"/>
 <wire x1="70.8" y1="55.88" x2="71.12" y2="55.56" width="0.4064" layer="1"/>
-<wire x1="54.29" y1="64.77" x2="57.15" y2="64.77" width="0.4064" layer="1"/>
 <wire x1="57.15" y1="64.77" x2="57.785" y2="64.135" width="0.4064" layer="1"/>
 <wire x1="70.485" y1="57.785" x2="71.12" y2="57.15" width="0.4064" layer="16"/>
@@
 <via x="58.42" y="63.5" extent="1-16" drill="0.6"/>
 <wire x1="58.42" y1="63.5" x2="57.785" y2="64.135" width="0.4064" layer="1"/>
+<contactref element="NOTA" pad="4"/>
+<wire x1="52.39" y1="67.57" x2="53.34" y2="68.52" width="0.4064" layer="1"/>
+<wire x1="53.34" y1="68.52" x2="57.15" y2="64.77" width="0" layer="19" extent="1-1"/>
 </signal>
 <signal name="N$4">
 <contactref element="IC4" pad="8"/>
-<contactref element="R7" pad="1"/>
 <contactref element="R21" pad="2"/>
 <wire x1="63.44" y1="55.88" x2="61.28" y2="55.88" width="0.4064" layer="1"/>
 <wire x1="61.28" y1="55.88" x2="60.96" y2="55.56" width="0.4064" layer="1"/>
-<wire x1="41.59" y1="64.77" x2="44.196" y2="64.77" width="0.4064" layer="1"/>
 <wire x1="44.196" y1="64.77" x2="45.72" y2="63.246" width="0.4064" layer="1"/>
 <wire x1="60.96" y1="55.56" x2="60.96" y2="57.15" width="0.4064" layer="1"/>
@@
 <wire x1="46.863" y1="58.293" x2="45.72" y2="59.436" width="0.4064" layer="1"/>
 <wire x1="45.72" y1="59.436" x2="45.72" y2="63.246" width="0.4064" layer="1"/>
+<contactref element="NOTB" pad="4"/>
+<wire x1="39.69" y1="67.57" x2="40.64" y2="68.52" width="0.4064" layer="1"/>
+<wire x1="44.196" y1="64.77" x2="40.64" y2="68.52" width="0" layer="19" extent="1-1"/>
 </signal>
 <signal name="N$5">
 <contactref element="IC4" pad="14"/>
-<contactref element="R10" pad="1"/>
 <contactref element="R26" pad="2"/>
 <wire x1="63.44" y1="48.26" x2="61.28" y2="48.26" width="0.4064" layer="1"/>
 <wire x1="61.28" y1="48.26" x2="60.96" y2="48.58" width="0.4064" layer="1"/>
-<wire x1="41.59" y1="52.07" x2="44.45" y2="52.07" width="0.4064" layer="1"/>
 <via x="65.532" y="48.26" extent="1-16" drill="0.6"/>
 <wire x1="65.532" y1="48.26" x2="63.44" y2="48.26" width="0.4064" layer="1"/>
@@
 <wire x1="61.849" y1="48.26" x2="65.532" y2="48.26" width="0.4064" layer="16"/>
 <wire x1="50.038" y1="54.61" x2="52.578" y2="52.07" width="0.4064" layer="16"/>
+<contactref element="VELB" pad="4"/>
+<wire x1="39.69" y1="54.87" x2="40.64" y2="55.82" width="0.4064" layer="1"/>
+<wire x1="40.64" y1="55.82" x2="44.45" y2="52.07" width="0" layer="19" extent="1-1"/>
 </signal>
 <signal name="N$25">
@@
 <wire x1="66.54" y1="54.11" x2="67.31" y2="53.34" width="0.3048" layer="1"/>
 <wire x1="67.31" y1="53.34" x2="68.64" y2="53.34" width="0.3048" layer="1"/>
-</signal>
-<signal name="N$31">
-<contactref element="R7" pad="2"/>
-<contactref element="NOTB" pad="4"/>
-<wire x1="39.69" y1="64.77" x2="39.69" y2="67.57" width="0.4064" layer="1"/>
-<wire x1="39.69" y1="67.57" x2="40.64" y2="68.52" width="0.4064" layer="1"/>
-</signal>
-<signal name="N$32">
-<contactref element="R10" pad="2"/>
-<contactref element="VELB" pad="4"/>
-<wire x1="39.69" y1="52.07" x2="39.69" y2="54.87" width="0.4064" layer="1"/>
-<wire x1="39.69" y1="54.87" x2="40.64" y2="55.82" width="0.4064" layer="1"/>
 </signal>
 <signal name="SR_DAT">
@@
 <wire x1="60.198" y1="76.708" x2="62.23" y2="78.74" width="0.4064" layer="16"/>
 </signal>
-<signal name="N$29">
-<contactref element="R11" pad="2"/>
-<contactref element="VELA" pad="4"/>
-<wire x1="52.39" y1="52.07" x2="52.39" y2="54.87" width="0.4064" layer="1"/>
-<wire x1="52.39" y1="54.87" x2="53.34" y2="55.82" width="0.4064" layer="1"/>
-</signal>
-<signal name="N$30">
-<contactref element="R8" pad="2"/>
-<contactref element="NOTA" pad="4"/>
-<wire x1="52.39" y1="64.77" x2="52.39" y2="67.57" width="0.4064" layer="1"/>
-<wire x1="52.39" y1="67.57" x2="53.34" y2="68.52" width="0.4064" layer="1"/>
-</signal>
 <signal name="N$38">
